File: OPA_POWER.kicad_sch (KiCad schematic)
At the start: 204 parts, among them J1 Conn_01x02, J10 Conn_02x14_Odd_Even, J11 Conn_01x04, J18 Conn_01x01, J19 Conn_01x01, J2 Jumper, J3 Jumper, J4 Jumper, J5 Jumper, J6 Jumper, J7 Jumper, J8 Jumper, J9 Conn_01x04, Q1 AO3400, Q2 AO3401, Q3 AO3400, Q4 AO3401, U1 XC6206, U10 LM337, U11 TPS7A2425, U12 TPS72325, U13 TPS7A39, U14 ADP7118(ADJ), U2 MP2333H, U3 ADP5071AREZ-R7, U4 LM2991S, U5 LM2940-9, U6 TPS7A30, U7 TPS7A49, U8 TPS65133, U9 LM317

Commit message: 更新預覽圖
Parts:
- C1, C29, C31: value Cap Pol1 -> 10uF
- C10, C14: value Cap -> 47nF
- C11: value Cap -> 1nF
- C12, C15, C16, C23, C25, C3, C39, C40, C57: value Cap -> 1uF
- C13: value Cap -> 6.8nF
- C19, C2, C20, C32, C33, C62: value Cap Pol1 -> Cap Pol1 10uF
- C21, C22, C28, C30, C34, C35, C36, C37, C50, C51, C6, C7, C8: value Cap -> 0.1uF
- C24: value Cap -> 10pF
- C26, C27, C5: value Cap Pol1 -> Cap Pol1 22uF
- C38, C41, C46, C47, C56, C58: value Cap -> 10nF
- C42, C43, C52, C53, C54, C55, C60, C63: value Cap Pol1 -> Cap Pol1 4.7uF
- C44, C45: value Tan -> Tan 10uF
- C48, C49: value Cap -> Cap NA
- C59, C61: value Cap -> 2.2uF
- L1, L2: value Inductor -> 2.2uH
- L3: value Inductor -> 10uH
- L4: value Inductor -> 0.47uH
- L7: value Inductor -> 4.7uH
- R1: value Res1 -> 200K
- R10, R31, R32, R9: value Res1 -> 20K
- R11, R39, R51, R58: value Res1 -> 10K
- R12: value Res1 -> 20R
- R13: value Res1 -> 7.68K
- R14, R17, R3, R35, R36: value Res1 -> 4.7K
- R15: value Res1 -> 40.2K
- R18: value Res1 -> 22K
- R19: value Res1 -> 2K
- R2, R20: value Res1 -> 100K
- R21: value Res1 -> 191K
- R22: value Res1 -> 250R
- R23, R42: value Res1 -> 30K
- R24: value Res1 -> 4R
- R25: value Res1 -> 4.42R
- R26, R27, R4, R6, R7: value Res1 -> 470K
- R28, R29, R33, R34, R57, R63, R64: value Res1 -> 0R
- R37: value Res1 -> 106R
- R40: value Res1 -> 3K
- R41: value Res1 -> 2.4K
- R45, R46, R47, R48, R49, R50: value Res1 -> NA
- R5: value Res1 -> 15K
- R52: value Res1 -> 40K
- R55: value Res1 -> 2.2K
- R56: value Res1 -> 32.4K
- R8: value Res1 -> 1K
Other:
- moved on the sheet: D10, D11, D12, D13, D14, D15, D16, D7, D8, D9, J10, J11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
