File: OPA_POWER_backup.kicad_pcb (KiCad board)
At the start: 4 copper layers, 110 x 80 mm, 205 parts, among them J1 Conn_01x02, J10 Conn_02x14_Odd_Even, J11 Conn_01x04, J18 Conn_01x01, J19 Conn_01x01, J2 Jumper, J3 Jumper, J4 Jumper, J5 Jumper, J6 Jumper, J7 Jumper, J8 Jumper, J9 Conn_01x04, Q1 AO3400, Q2 AO3401, Q3 AO3400, Q4 AO3401, U1 XC6206, U10 LM337, U11 TPS7A2425, U12 TPS72325, U13 TPS7A39, U14 ADP7118(ADJ), U2 MP2333H, U3 ADP5071AREZ-R7, U4 LM2991S, U5 LM2940-9, U6 TPS7A30, U7 TPS7A49, U8 TPS65133, U9 LM317

Commit message: 更新預覽圖
Parts:
- removed REF**: KiCad-Logo_30mm_SilkScreen, Symbol:KiCad-Logo_30mm_SilkScreen
Other:
- board text added: "+20V"
- board text added: "+5.0V"
- board text added: "+9.0V"
- board text added: "-20V"
- board text added: "-5.0V"
- board text added: "-9.0V"
- board text added: "D3.3V"
- board text added: "D5.0V"
- board text added: "VER 1.0 202306"
